Commit message: Version final de las diapositivas y ejercicios

File: catkin_ws/src/hardware/justina_description/urdf/justina_base.xacro (robot description, xacro)
@@ -206,5 +206,5 @@
   </link>
   <joint name="laser_connect" type="fixed">
-    <origin xyz="0.17 0 0.44" />
+    <origin xyz="0.17 0 0.44" rpy="0 0 0"/>
     <parent link="base_link"/>
     <child link="laser_link"/>
